File: Bell-AY-3-8910.kicad_pcb (KiCad board)
At the start: 2 copper layers, 90 x 83 mm, 33 parts, among them U1 8085, U2 27C256, U3 ATF16V, U4 HM6116, U5 74LS573, U6 AY-3-8910, Y1 3.54Mhz

Commit message: 1
Parts:
- removed BELL: SW3, Button_Switch_THT:SW_PUSH_6mm
- removed DOOR: SW2, Connector_JST:JST_EH_B2B-EH-A_1x02_P2.50mm_Vertical
- removed PWR: J1, Connector_JST:JST_EH_B2B-EH-A_1x02_P2.50mm_Vertical
- removed RESET: SW1, Button_Switch_THT:SW_Tactile_SPST_Angled_PTS645Vx39-2LFS
- removed SPEAK: J2, Connector_JST:JST_EH_B2B-EH-A_1x02_P2.50mm_Vertical
- added BELL1: SW3, Button_Switch_THT:SW_PUSH_6mm, F.Cu at (119.0, 96.0)
- added DOOR1: SW2, Connector_JST:JST_EH_B2B-EH-A_1x02_P2.50mm_Vertical, F.Cu at (150.0, 93.0)
- added PWR1: J1, Connector_JST:JST_EH_B2B-EH-A_1x02_P2.50mm_Vertical, F.Cu at (154.0, 21.0)
- added RESET1: SW1, Button_Switch_THT:SW_Tactile_SPST_Angled_PTS645Vx39-2LFS, F.Cu at (28.0, 23.0)
- added SPEAK1: J2, Connector_JST:JST_EH_B2B-EH-A_1x02_P2.50mm_Vertical, F.Cu at (150.0, 99.0)
- moved C3 120.2 mm to (142.0, 21.0)
- moved C6 94.6 mm to (162.0, 81.0), turned to 0 degrees
- moved C8 93.0 mm to (162.0, 90.0), turned to 0 degrees
- moved R5 89.0 mm to (131.0, 88.0)
- moved R4 89.0 mm to (131.0, 92.0)
- moved R3 89.0 mm to (131.0, 96.0)
- moved R2 89.0 mm to (131.0, 100.0)
- moved H4 85.0 mm to (23.0, 100.0)
- moved H2 82.1 mm to (105.0, 23.0)
- moved H1 77.3 mm to (23.0, 23.0)
- moved H3 77.2 mm to (105.0, 100.0)
- moved C5 65.3 mm to (162.0, 76.0), turned to 0 degrees
- moved C7 59.7 mm to (162.0, 85.0), turned to 0 degrees
- moved C9 56.8 mm to (162.0, 95.0), turned to 0 degrees
- moved C10 54.9 mm to (162.0, 100.0), turned to 0 degrees
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